Commit message: move left control to finger tip

File: pink_backend/panda_blender_left.urdf (robot description, URDF)
Before this commit: robot panda_blender_left, 11 links, 10 joints
Links:
- added link fer_leftfinger
- added link fer_rightfinger
- added link tcp_fingertips
Joints:
- added joint fer_finger_joint1: type fixed, parent fer_hand, child fer_leftfinger, origin xyz=0 0 0.0584 rpy=0 0 0
- added joint fer_finger_joint2: type fixed, parent fer_hand, child fer_rightfinger, origin xyz=0 0 0.0584 rpy=0 0 0
- added joint tcp_fingertips_joint: type fixed, parent fer_hand, child tcp_fingertips, origin xyz=0 0 0.1034 rpy=0 0 0
