Commit message: move right arm tcp to finger tip

File: pink_backend/panda_blender_right.urdf (robot description, URDF)
Before this commit: robot panda_blender_right, 11 links, 10 joints
Links:
- added link fer_leftfinger
- added link fer_rightfinger
- added link fer_sensone
- added link tcp_fingertips
Joints:
- added joint fer_finger_joint1: type fixed, parent fer_hand, child fer_leftfinger, origin xyz=0 0.0584 0 rpy=0 0 0
- added joint fer_finger_joint2: type fixed, parent fer_hand, child fer_rightfinger, origin xyz=0 0.0584 0 rpy=0 0 0
- added joint fer_sensone_joint: type fixed, parent fer_link8, child fer_sensone, origin xyz=-0.0021109185 0.0379412062 0.0000948205 rpy=-0.6154799466 -0.5235987285 0.9553164954
- added joint tcp_fingertips_joint: type fixed, parent fer_hand, child tcp_fingertips, origin xyz=0 0.1034 0 rpy=0 0 0
- joint fer_hand_joint: origin xyz=-0.0021109185 0.0379412062 0.0000948205 rpy=-0.0000002226 -0.7853983045 -0.0000000843 -> xyz=0 0 0 rpy=0 0 -0.785398163397; parent fer_link8 -> fer_sensone
